File: elec/layout/default/benou-75board.kicad_pcb (KiCad board)
At the start: 2 copper layers, 225.7 x 100.8 mm, 0 parts

Commit message: Initial RP2040 kit
Parts:
- added C1: 22.0 pF, lib:C0402, F.Cu at (55.8, -31.6)
- added C10: 100.0 nF, lib:C0402, F.Cu at (44.5, -12.1)
- added C11: 100.0 nF, lib:C0402, F.Cu at (65.6, -31.6)
- added C12: 1.0 uF, lib:C0402, F.Cu at (60.7, -35.6)
- added C2: 22.0 pF, lib:C0402, F.Cu at (65.5, -24.4)
- added C3: 100.0 nF, lib:C0402, F.Cu at (65.5, -16.4)
- added C4: 100.0 nF, lib:C0402, F.Cu at (65.5, -12.4)
- added C5: 100.0 nF, lib:C0402, F.Cu at (60.7, -31.6)
- added C6: 100.0 nF, lib:C0402, F.Cu at (55.8, -35.6)
- added C7: 100.0 nF, lib:C0402, F.Cu at (60.6, -12.4)
- added C8: 1.0 uF, lib:C0402, F.Cu at (65.6, -35.6)
- added C9: 100.0 nF, lib:C0402, F.Cu at (65.5, -20.4)
- added R1: 1.0 KΩ, lib:R0402, F.Cu at (53.2, -13.7)
- added R2: 27.0 KΩ, lib:R0402, F.Cu at (60.6, -16.4)
- added R3: 27.0 KΩ, lib:R0402, F.Cu at (60.6, -20.4)
- added R4: 10.0 KΩ, lib:R0402, F.Cu at (60.6, -24.4)
- added R5: 10.0 KΩ, lib:R0402, F.Cu at (53.2, -17.6)
- added U1: , lib:LQFN-56_L7.0-W7.0-P0.4-EP, F.Cu at (47.8, -31.9)
- added U2: , lib:OSC-SMD_4P-L3.2-W2.5-BL, F.Cu at (54.6, -23.1)
- added U3: , lib:SOIC-8_L5.3-W5.3-P1.27-LS8.0-BL, F.Cu at (46.5, -20.2)
Other:
- board size 225.7 x 100.8 mm -> 40 x 40 mm
